File: meshtastic-build-off-2026/Hardware/Untitled/lora.kicad_sch (KiCad schematic)
At the start: 2 parts, among them U4 Wio-SX1262

Commit message: Working DRC
Connections:
- net SPI_MISO renamed SPI_MISO_LORA
- net SPI_MOSI renamed SPI_MOSI_LORA
- net SPI_SCK renamed SPI_SCK_LORA
Changed lines of the file:
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@@
 		)
 	)
-	(hierarchical_label "SPI_MOSI"
+	(hierarchical_label "SPI_MOSI_LORA"
 		(shape input)
 		(at 97.79 66.04 180)
@@
 		)
 	)
-	(hierarchical_label "SPI_SCK"
+	(hierarchical_label "SPI_SCK_LORA"
 		(shape input)
 		(at 97.79 68.58 180)
@@
 		)
 	)
-	(hierarchical_label "SPI_MISO"
+	(hierarchical_label "SPI_MISO_LORA"
 		(shape input)
 		(at 97.79 63.5 180)
