File: meshtastic-build-off-2026/Hardware/Untitled/mcu_core.kicad_sch (KiCad schematic)
At the start: 6 parts, among them SW1 SW_Push, U1 ESP32-S3-WROOM-1

Commit message: Working DRC
Connections:
- net DISPLAY_CS: now also U1.5 (IO5); no longer U1.17 (IO9)
- net KB_C2: now also U1.38 (IO2); no longer U1.23 (IO21)
- net KB_C3: now also U1.39 (IO1); no longer U1.24 (IO47)
- net LORA_CS: now also U1.17 (IO9); no longer U1.18 (IO10)
- net LORA_DI01: now also U1.23 (IO21); no longer U1.8 (IO15)
- net LORA_DI02: now also U1.22 (IO14); no longer U1.9 (IO16)
- net LORA_RST: now also U1.18 (IO10); no longer U1.7 (IO7)
- net TFT_BL: now also U1.4 (IO4); no longer U1.6 (IO6)
- net TFT_DC: now also U1.6 (IO6); no longer U1.4 (IO4)
- net TFT_RST: now also U1.7 (IO7); no longer U1.5 (IO5)
- net SPI_MISO renamed SPI_MISO_LORA
- net SPI_MOSI renamed SPI_MOSI_LORA
- net SPI_SCK renamed SPI_SCK_LORA
- new net TFT_MOSI: U1.8 (IO15)
- new net TFT_SCK: U1.9 (IO16)

Commit message: updated PCB
Parts:
- SW1: footprint Button_Switch_SMD:SW_Push_1P1T_NO_CK_KSC6xxJ -> Button_Switch_SMD:SW_SPST_Omron_B3FS-100xP
Connections:
- net KB_C1: now also U1.25 (IO48); no longer U1.35 (IO42)
- net KB_C2: now also U1.39 (IO1); no longer U1.38 (IO2)
- net KB_C3: now also U1.38 (IO2); no longer U1.39 (IO1)
- net KB_C4: now also U1.35 (IO42); no longer U1.25 (IO48)
- net LORA_CS: now also U1.23 (IO21); no longer U1.17 (IO9)
- net LORA_DI01: now also U1.17 (IO9); no longer U1.23 (IO21)
- net LORA_DI02: now also U1.18 (IO10); no longer U1.22 (IO14)
- net LORA_RST: now also U1.22 (IO14); no longer U1.18 (IO10)
- net SPI_MISO_LORA: now also U1.19 (IO11); no longer U1.21 (IO13)
- net SPI_SCK_LORA: now also U1.21 (IO13); no longer U1.19 (IO11)
