File: meshtastic-build-off-2026/Hardware/meshtalk_t9/lora.kicad_sch (KiCad schematic)
At the start: 2 parts, among them U4 Wio-SX1262

Commit message: rename + battery % + boot btn changed to reset + fix battery chrging
Changed lines of the file:
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@@
 	(paper "A4")
 	(junction
-		(at 85.09 76.2)
+		(at 96.52 78.74)
 		(diameter 0)
 		(color 0 0 0 0)
 	)
 	(junction
-		(at 96.52 78.74)
+		(at 85.09 76.2)
 		(diameter 0)
 		(color 0 0 0 0)
@@
 		(pts
 			(xy 102.87 66.0908) (xy 102.87 67.31)
-		)
-		(stroke
-			(width 0)
-			(type default)
-		)
-	)
-	(wire
-		(pts
-			(xy 85.09 78.74) (xy 85.09 76.2)
 		)
 		(stroke
@@
 		)
 		(stroke
+			(width 0)
+			(type default)
+		)
+	)
+	(wire
+		(pts
+			(xy 85.09 76.2) (xy 85.09 78.74)
+		)
+		(stroke

Commit message: Replace AP2112K-3.3  with AP7361C-33E Connected LORA RF_SW1 to GPIO Added ESD Added mounting holes for display (Waveshare 2 inch) Added Boot and Reset buttons made power rails thicker added dedicated layer for 3v3 and GND
Parts:
- C6: MPN (none) -> CC0805KRX7R9BB104; Manufacturer (none) -> YAGEO
- U4: MPN (none) -> Wio-SX1262
Connections:
- net GND: now also U4.10 (GND2)
- net LORA_RF_SW1: now reaches U4.1 (RF_SW1)
- net LORA_DI02 renamed LORA_BUSY
Changed lines of the file:
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@@
+	(wire
+		(pts
+			(xy 128.2192 68.58) (xy 132.08 68.58)
+		)
+		(stroke
+			(width 0)
+			(type default)
+		)
+	)
 	(wire
 		(pts
@@
 	(wire
 		(pts
+			(xy 96.52 60.96) (xy 102.87 60.96)
+		)
+		(stroke
+			(width 0)
+			(type default)
+		)
+	)
+	(wire
+		(pts
 			(xy 102.87 71.12) (xy 97.79 71.12)
 		)
@@
 	(wire
 		(pts
+			(xy 128.2192 68.58) (xy 128.2192 68.6054)
+		)
+		(stroke
+			(width 0)
+			(type default)
+		)
+	)
+	(wire
+		(pts
 			(xy 97.79 69.85) (xy 97.79 68.58)
 		)
@@
 	(wire
 		(pts
+			(xy 102.87 60.96) (xy 102.87 61.0108)
+		)
+		(stroke
+			(width 0)
+			(type default)
+		)
+	)
+	(wire
+		(pts
 			(xy 132.08 63.5508) (xy 132.08 63.5)
 		)
@@
 		)
 	)
+	(hierarchical_label "LORA_RF_SW1"
+		(shape input)
+		(at 96.52 60.96 180)
+		(effects
+			(font
+				(size 1.27 1.27)
+			)
+			(justify right)
+		)
+	)
 	(hierarchical_label "LORA_RST"
 		(shape input)
@@
 		)
 	)
-	(hierarchical_label "LORA_DI02"
+	(hierarchical_label "LORA_BUSY"
 		(shape input)
 		(at 132.08 66.04 0)
@@
 			)
 		)
+		(property "MPN" "Wio-SX1262"
+			(at 115.57 69.85 0)
+			(effects
+				(font
+					(size 1.27 1.27)
+				)
+				(hide yes)
+			)
+		)
 		(pin "9"
 		)
@@
 			)
 		)
+		(property "MPN" "CC0805KRX7R9BB104"
+			(at 88.9 78.74 90)
+			(effects
+				(font
+					(size 1.27 1.27)
+				)
+				(hide yes)
+			)
+		)
+		(property "Manufacturer" "YAGEO"
+			(at 88.9 78.74 90)
+			(effects
+				(font
+					(size 1.27 1.27)
+				)
+				(hide yes)
+			)
+		)
 		(pin "2"
 		)
@@
 					(unit 1)
 				)
+			)
+		)
+	)
+	(symbol
+		(lib_id "power:GND")
+		(at 132.08 68.58 90)
+		(unit 1)
+		(exclude_from_sim no)
+		(in_bom yes)
+		(on_board yes)
+		(dnp no)
+		(fields_autoplaced yes)
+		(property "Reference" "#PWR017"
+			(at 138.43 68.58 0)
+			(effects
+				(font
+					(size 1.27 1.27)
+				)
+				(hide yes)
+			)
+		)
+		(property "Value" "GND"
+			(at 135.89 68.5799 90)
+			(effects
+				(font
+					(size 1.27 1.27)
+				)
+				(justify right)
+			)
+		)
+		(property "Footprint" ""
+			(at 132.08 68.58 0)
+			(effects
+				(font
+					(size 1.27 1.27)
+				)
+				(hide yes)
+			)
+		)
+		(property "Datasheet" ""
+			(at 132.08 68.58 0)
+			(effects
+				(font
+					(size 1.27 1.27)
+				)
+				(hide yes)
+			)
+		)
+		(property "Description" "Power symbol creates a global label with name \"GND\" , ground"
+			(at 132.08 68.58 0)
+			(effects
+				(font
+					(size 1.27 1.27)
+				)
+				(hide yes)
+			)
+		)
+		(pin "1"
+		)
+		(instances
+			(project ""
+				(path "/81d8a60b-fb85-4750-b4ba-90a418a69e1e/00cd80e2-981f-4300-9615-3109ca1a0085"
+					(reference "#PWR017")
+					(unit 1)
+				)
