File: meshtastic-build-off-2026/Hardware/meshtalk_t9/meshtalk_t9.kicad_pcb (KiCad board)
At the start: 4 copper layers, 60.2 x 79.2 mm, 60 parts, among them J1 USB_C_Receptacle_USB2.0_16P, J2 Conn_01x02_Socket, Q1 Q_PMOS_GSD, Q2 2N7002, Q3 Q_PMOS_GSD, SW1 SW_Push, SW10 SW_Push, SW11 SW_Push, SW12 SW_Push, SW13 SW_Push, SW14 SW_Push, SW15 SW_Push, SW16 SW_Push, SW17 SW_Push, SW18 SW_Push, SW2 SW_Push, SW3 SW_Push, SW4 SW_Push, SW5 SW_Push, SW6 SW_Push, SW7 SW_Push, SW8 SW_Push, SW9 SW_Push, U1 ESP32-S3-WROOM-1, U2 USBLC6-2SC6, U3 MCP73831-2-MC, U4 Wio-SX1262, U5 AP7361C-33E

Commit message: add T9 configurations for meshtastic
Parts:
- moved J1 1.85 mm to (59.7, 37.5), turned to 180 degrees
Routing:
- net Net-(D1-A): track 52.6 -> 62.2 mm
- net Net-(J1-D+-PadA6): track 19.4 -> 12.7 mm
- net Net-(J1-D--PadA7): track 19.9 -> 15.7 mm, vias 2 -> 0
- net GND: track 129.0 -> 132.9 mm, vias 21 -> 22
- net Net-(J1-CC2): track 18.4 -> 14.6 mm
- net Net-(J1-CC1): track 9.34 -> 13.0 mm, vias 0 -> 2
